Commit message: Trying to debug why the locate function is not returning the right data. It looks like the distances are fine but the angle is following the torsofront2back?

File: backend/Testing/FullAssem11_24_23(1).urdf (robot description, URDF)
Before this commit: robot FullAssem11_25_23, 28 links, 27 joints
Joints:
- joint HipsSide2Side: axis 0 0 1 -> 0 0 -1
